Commit message: refresh

File: indy7_description/urdf/gripper_3f.xacro (robot description, xacro)
@@ -1,5 +1,5 @@
 <?xml version="1.0" ?>
 <robot name="gripper" xmlns:xacro="http://ros.org/wiki/xacro">
-  <xacro:include filename="$(find robotiq_3f_description)/urdf/robotiq-3f-gripper_articulated.xacro"/>
+  <xacro:include filename="$(find robotiq_3f_description)/urdf/robotiq-3f-gripper_articulated.xacro" />
  <!-- verificar angulo de support_gripper -->
   <link name="support_gripper_link">
@@ -43,5 +43,5 @@
     <origin rpy="0 0 0" xyz="0 0 0.008"/>
   </joint>
-  <joint name="indy7_support_gripper" type="fixed">
+  <joint name="indy7_joint_gripper" type="fixed">
     <parent link="support_gripper_link"/>
     <child link="palm"/>

File: indy7_description/urdf/indy7.urdf (robot description, URDF)
Before this commit: robot indy7, 9 links, 8 joints
Links:
- link link0: geometry visual mesh filename=package://indy7_description/meshes/indy7/Indy7_0.
