Commit message: update

File: indy7_description/urdf/gripper_2f.xacro (robot description, xacro)
@@ -50,6 +50,6 @@
   <!-- end effect point -->
   <joint name="end_effect_point" type="fixed">
-    <origin rpy="0 0 0" xyz="0 0 0.15"/>
-    <parent link="support_gripper_link"/>
+    <origin rpy="0 0 0" xyz="0 0 0.17"/>
+    <parent link="tcp"/>
     <child link="end_effect_point"/>
   </joint>

File: indy7_description/urdf/gripper_3f.xacro (robot description, xacro)
@@ -51,5 +51,5 @@
   <joint name="end_effect_point" type="fixed">
     <origin rpy="0 0 0" xyz="0 0 0.15"/>
-    <parent link="support_gripper_link"/>
+    <parent link="tcp"/>
     <child link="end_effect_point"/>
   </joint>

File: indy7_description/urdf/indy7.urdf (robot description, URDF)
Before this commit: robot indy7, 9 links, 8 joints
Links:
- link link0: geometry visual mesh filename=package://indy7_description/meshes/indy7/Indy7_0.stl
